File: falling-shapes-earrings/falling-shapes-earrings.kicad_sch (KiCad schematic)
At the start: 28 parts, among them U1 ATTINY85-20SUR

Commit message: Update falling-shapes-earrings.kicad_sch
V0.1
Parts:
- XBT1: footprint (none) -> Power Management:SMTU1632LF; PART_NUMBER SMTU1632-LF -> 701130
Changed lines of the file:
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@@
 		(title "Falling Shapes Earrings")
 		(date "2026-04-07")
-		(rev "v.0.03")
+		(rev "v.0.10")
 		(company "Tottocs")
 	)
@@
 		)
 		(property "Value" "GNDREF"
-			(at 97.79 90.17 0)
+			(at 97.79 88.9 0)
 			(hide yes)
 			(show_name no)
@@
 		)
 		(property "Value" "GNDREF"
-			(at 120.65 90.17 0)
+			(at 120.65 88.9 0)
 			(hide yes)
 			(show_name no)
@@
 			)
 		)
-		(property "Footprint" ""
+		(property "Footprint" "Power Management:SMTU1632LF"
 			(at 27.94 34.29 0)
 			(hide yes)
@@
 			)
 		)
-		(property "PART_NUMBER" "SMTU1632-LF"
+		(property "PART_NUMBER" "701130"
 			(at 27.94 34.29 0)
 			(hide yes)
@@
 		)
 		(property "Value" "GNDREF"
-			(at 143.51 90.17 0)
+			(at 143.51 88.9 0)
 			(hide yes)
 			(show_name no)
@@
 		)
 		(property "Value" "GNDREF"
-			(at 25.4 78.74 0)
+			(at 25.4 77.47 0)
 			(hide yes)
 			(show_name no)
@@
 		)
 		(property "Value" "GNDREF"
-			(at 165.1 90.17 0)
+			(at 165.1 88.9 0)
 			(hide yes)
 			(show_name no)
